File: wearable/pcb/wearable-core.kicad_sch (KiCad schematic)
At the start: 62 parts, among them J1 USB_C_Receptacle_USB2.0, J2 Extension, U1 BC833, U2 MCP73832-2-OT, U3 S-85S1A, U4 LIS2DE12, U5 APDS-9250, U6 MX25R8035FZxxx0, U7 PCF85063ATL, U8 DT1446-04V, Y71 32.768kHz

Commit message: Part of #16. Added GNSS PCB layout
Also added custom footprint for NN02-224 chip antenna.
Signed-off-by: Adam Fowler <adam@adamfowler.org>
Parts:
- FB1, FB2: symbol Device:Ferrite_Bead -> Device:FerriteBead
Connections:
- net Earth: now also FB1.1
- net GND: now also FB1.2, FB2.2
- net GNDPWR: now also FB2.1
- no-connect marks 9 -> 8
Changed lines of the file:
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@@
   (junction (at 38.1 144.78) (diameter 0) (color 0 0 0 0)
   )
-  (junction (at 137.16 149.86) (diameter 0) (color 0 0 0 0)
-  )
   (junction (at 158.75 162.56) (diameter 0) (color 0 0 0 0)
   )
@@
   (junction (at 76.2 21.59) (diameter 0) (color 0 0 0 0)
   )
-  (no_connect (at 137.16 147.32))
   (no_connect (at 76.2 53.34))
   (no_connect (at 53.34 49.53))
@@
     (stroke (width 0) (type default))
   )
-  (wire (pts (xy 123.19 149.86) (xy 137.16 149.86))
+  (wire (pts (xy 123.19 149.86) (xy 142.24 149.86))
     (stroke (width 0) (type default))
   )
@@
     (stroke (width 0) (type default))
   )
-  (wire (pts (xy 137.16 149.86) (xy 142.24 149.86))
-    (stroke (width 0) (type default))
-  )
   (wire (pts (xy 154.94 154.94) (xy 158.75 154.94))
     (stroke (width 0) (type default))
@@
   )
   (wire (pts (xy 256.54 45.72) (xy 254 45.72))
-    (stroke (width 0) (type default))
-  )
-  (wire (pts (xy 137.16 147.32) (xy 137.16 149.86))
     (stroke (width 0) (type default))
   )
@@
     )
   )
-  (symbol (lib_id "Device:Ferrite_Bead") (at 30.48 63.5 0) (unit 1)
+  (symbol (lib_id "Device:FerriteBead") (at 30.48 63.5 0) (unit 1)
     (in_bom yes) (on_board yes) (dnp no)
     (property "Reference" "FB1" (at 27.0256 62.3316 0)
@@
       (effects (font (size 1.27 1.27)) hide)
     )
+    (pin "1")
+    (pin "2")
     (instances
       (project "wearable"
@@
     )
   )
-  (symbol (lib_id "Device:Ferrite_Bead") (at 38.1 63.5 0) (unit 1)
+  (symbol (lib_id "Device:FerriteBead") (at 38.1 63.5 0) (unit 1)
     (in_bom yes) (on_board yes) (dnp no)
     (property "Reference" "FB2" (at 41.5798 62.3316 0)
@@
       (effects (font (size 1.27 1.27)) hide)
     )
+    (pin "1")
+    (pin "2")
     (instances
       (project "wearable"
