File: wearable-v2/pcb/wearable-v2.kicad_pcb (KiCad board)
At the start: 2 copper layers, 112.1 x 40.2 mm, 109 parts, among them IC1 TESEO-LIV3F, J1 HERALD_V2_CONN_RECEPTACLE, J16 EA_WF030-39S, J17 JST_AUDIO_OUT, J18 DEBUG_HERALD, J19 FTDI_HERALD, J2 HERALD_V2_CONN_RECEPTACLE, J3 HERALD_V2_CONN_RECEPTACLE, J4 HERALD_V2_CONN_RECEPTACLE, J5 HERALD_V2_CONN_PORT, J6 HERALD_V2_CONN_PORT, J7 USB_C_Receptacle_USB2.0, J8 HERALD_V2_CONN_PORT, J9 HERALD_V2_CONN_PORT, SW1 SW_Push, U1 DT1446-04V, U10 ATmega328PB-M, U11 TMP1075, U12 MAX30102, U13 TPA6139A2RGTR, U14 LIS2DE12, U15 TLV751, U16 DRV2605LDGS, U2 MCP73831/2-2MC, U3 TCA6408A, U4 FT201XQ, U5 MX25R6435FZNIL0, U6 BC833, U7 MX25R6435F, U8 PCF85063ATL, U9 APDS-9250, Y1 32.768kHz, Y2 8Mhz

Commit message: Split main boards out into their own KiCAD files
Signed-off-by: Adam Fowler <adam@adamfowler.org>
Parts:
- added BoardBio: Board Bio, PCM_kikit:Board, F.Cu at (163.6, 99.1)
- added BoardFeedback: Board Feedback, PCM_kikit:Board, F.Cu at (144.8, 124.2)
- added BoardPositioning: Board Positioning, PCM_kikit:Board, F.Cu at (107.3, 121.5)
- added ComputeBC833M: Board Compute BC833M, PCM_kikit:Board, F.Cu at (119.5, 99.2)
- added ConnectorStandard: Board Standard Connector, PCM_kikit:Board, F.Cu at (98.7, 99.1)
- added PanelAmbientLight: Board Ambient Light Panel, PCM_kikit:Board, F.Cu at (67.1, 99.1)
- added PanelButton: Board Button Panel, PCM_kikit:Board, F.Cu at (81.2, 127.1)
